Commit message: corrected the urdf

File: install/dumme_description/share/dumme_description/urdf/dumme_description.urdf.xacro (robot description, xacro)
@@ -209,5 +209,5 @@
     <!-- Adjust this position -->
     <origin xyz="-2.2 0 6.6" rpy="0 0 0"/>
-    <parent link="base_joint"/>
+    <parent link="base"/>
     <child link="camera_mount"/>
   </joint>

Commit message: movit configured

File: install/dumme_description/share/dumme_description/urdf/dumme_description.urdf.xacro (robot description, xacro)
@@ -73,5 +73,5 @@
           lower="-3.14159"
           upper="3.14159"
-          effort="100"
+          effort="10000"
           velocity="1"/>
       </joint>
@@ -109,5 +109,5 @@
           lower="-3.14159"
           upper="3.14159"
-          effort="100"
+          effort="10000"
           velocity="1"/>
       </joint>
@@ -145,5 +145,5 @@
           lower="-3.14159"
           upper="3.14159"
-          effort="100"
+          effort="10000"
           velocity="1"/>
       </joint>
@@ -177,5 +177,5 @@
     <child link="wrist"/>
     <axis xyz="0.47573 -0.87959 0.0026889"/>
-    <limit lower="-3.14159" upper="3.14159" effort="100" velocity="1"/>
+    <limit lower="-3.14159" upper="3.14159" effort="10000" velocity="1"/>
   </joint>
   <!-- ================= CAMERA MOUNT ================= -->
